File: PCB/FPGA_PPU.sch (EAGLE design)
At the start: 103 parts, among them CON1 DIP40, J1 J-08-SIP-100, T1 BC847, U1 74LVC4245APW,112, U2 74LVC4245APW,112, U3 SN74LVC541A, U4 ADV7125KST140, U5 THS7374IPWR, U6 EPCS4, U7 SN74LVC1G17DBVR, U8 EP2C5T144, X1 057-010-1

Commit message: Add files via upload
Connections:
- net +3V3: now also U6.VCC@2, U6.VCC@3; no longer U6.VCC2@2, U6.VCC3@3
Changed lines of the file:
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@@
 <part name="GND73" library="supply1" library_urn="urn:adsk.eagle:library:371" deviceset="GND" device=""/>
 <part name="C46" library="SnapEDA-Library" deviceset="ELCAP" device="" value="22uF"/>
-<part name="U6" library="EPCS4" deviceset="EPCS4" device=""/>
 <part name="V1" library="supply" deviceset="+1V2" device=""/>
 <part name="V2" library="supply" deviceset="+1V2" device=""/>
@@
 <part name="J1" library="con-headers-jp" deviceset="J-08-" device="SIP-100"/>
 <part name="CON1" library="SnapEDA-Library" deviceset="DIP40" device=""/>
+<part name="U6" library="EPCS4" deviceset="EPCS4" device=""/>
 </parts>
 <sheets>
@@
 <attribute name="VALUE" x="-102.67" y="-121.24" size="1.778" layer="96"/>
 </instance>
-<instance part="U6" gate="G$1" x="182.88" y="0" smashed="yes">
-<attribute name="NAME" x="181.757" y="8.422659375" size="1.77853125" layer="95"/>
-<attribute name="VALUE" x="177.7856" y="-7.63081875" size="1.78051875" layer="96"/>
-</instance>
 <instance part="V1" gate="G$1" x="132.08" y="109.22" smashed="yes">
 <attribute name="VALUE" x="128.905" y="111.76" size="1.778" layer="96"/>
@@
 <attribute name="VALUE" x="-77.1" y="2.53" size="1.778" layer="96"/>
 </instance>
+<instance part="U6" gate="G$1" x="182.88" y="0" smashed="yes">
+<attribute name="NAME" x="181.507" y="8.492659375" size="1.77853125" layer="95"/>
+<attribute name="VALUE" x="179.0156" y="-7.69081875" size="1.78051875" layer="96"/>
+</instance>
 </instances>
 <busses>
@@
 <wire x1="200.66" y1="12.7" x2="198.12" y2="12.7" width="0.1524" layer="91"/>
 <junction x="198.12" y="12.7"/>
-<pinref part="U6" gate="G$1" pin="VCC2@2"/>
-<pinref part="U6" gate="G$1" pin="VCC3@3"/>
-<pinref part="U6" gate="G$1" pin="VCC@1"/>
 <pinref part="V14" gate="G$1" pin="+3V3"/>
+<pinref part="U6" gate="G$1" pin="VCC@2"/>
+<pinref part="U6" gate="G$1" pin="VCC@3"/>
+<pinref part="U6" gate="G$1" pin="VCC@1"/>
 </segment>
 <segment>

Commit message: Add files via upload
Parts:
- U1, U2: value 74LVC4245APW,112 -> SN74LVC8T245; device SnapEDA-Library:74LVC4245APW,112 -> SnapEDA-Library:SN74LVC8T245
Connections:
- net /DBE_FPGA: now also U2./OE; no longer U1.~OE
- net /PRD: now also U1.DIR; no longer U2.DIR
- net D0_FPGA: now also U2.A0; no longer U1.A0
- net D1_FPGA: now also U2.A1; no longer U1.A1
- net D2_FPGA: now also U2.A2; no longer U1.A2
- net D3_FPGA: now also U2.A3; no longer U1.A3
- net D4_FPGA: now also U2.A4; no longer U1.A4
- net D5_FPGA: now also U2.A5; no longer U1.A5
- net D6_FPGA: now also U2.A6; no longer U1.A6
- net D7_FPGA: now also U2.A7; no longer U1.A7
- net DB0: now also U2.B0; no longer U1.B0
- net DB1: now also U2.B1; no longer U1.B1
- net DB2: now also U2.B2; no longer U1.B2
- net DB3: now also U2.B3; no longer U1.B3
- net DB4: now also U2.B4; no longer U1.B4
- net DB5: now also U2.B5; no longer U1.B5
- net DB6: now also U2.B6; no longer U1.B6
- net DB7: now also U2.B7; no longer U1.B7
- net PD0: now also U1.B0; no longer U2.B0
- net PD0_FPGA: now also U1.A0; no longer U2.A0
- net PD1: now also U1.B1; no longer U2.B1
- net PD1_FPGA: now also U1.A1; no longer U2.A1
- net PD2: now also U1.B2; no longer U2.B2
- net PD2_FPGA: now also U1.A2; no longer U2.A2
- net PD3: now also U1.B3; no longer U2.B3
- net PD3_FPGA: now also U1.A3; no longer U2.A3
- net PD4: now also U1.B4; no longer U2.B4
- net PD4_FPGA: now also U1.A4; no longer U2.A4
- net PD5: now also U1.B5; no longer U2.B5
- net PD5_FPGA: now also U1.A5; no longer U2.A5
- net PD6: now also U1.B6; no longer U2.B6
- net PD6_FPGA: now also U1.A6; no longer U2.A6
- net PD7: now also U1.B7; no longer U2.B7
- net PD7_FPGA: now also U1.A7; no longer U2.A7
- net PD_OE: now also U1./OE; no longer U2.~OE
- net RW_FPGA: now also U2.DIR; no longer U1.DIR

Commit message: Add files via upload
Parts:
- R10: value 1k -> 910
- R11: value 75R -> 75
- R15: value 10k -> 1.1k
- R16: value 10k -> 510
Other:
- note added: "EXT LSB ADDRESS DATA"
Changed lines of the file:
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@@
 <?xml version="1.0" encoding="utf-8"?>
 <!DOCTYPE eagle SYSTEM "eagle.dtd">
-<eagle version="9.6.2">
+<eagle version="9.4.2">
 <drawing>
 <settings>
@@
 <setting verticaltext="up"/>
 </settings>
-<grid distance="0.1" unitdist="inch" unit="inch" style="lines" multiple="1" display="yes" altdistance="0.01" altunitdist="mm" altunit="mm"/>
+<grid distance="0.1" unitdist="inch" unit="inch" style="lines" multiple="1" display="yes" altdistance="0.000393700787" altunitdist="inch" altunit="inch"/>
 <layers>
 <layer number="1" name="Top" color="4" fill="1" visible="no" active="no"/>
@@
 <part name="GND7" library="supply1" library_urn="urn:adsk.eagle:library:371" deviceset="GND" device=""/>
 <part name="GND8" library="supply1" library_urn="urn:adsk.eagle:library:371" deviceset="GND" device=""/>
-<part name="R10" library="rcl" library_urn="urn:adsk.eagle:library:334" deviceset="R-EU_" device="R0805" package3d_urn="urn:adsk.eagle:package:23553/2" value="1k"/>
+<part name="R10" library="rcl" library_urn="urn:adsk.eagle:library:334" deviceset="R-EU_" device="R0805" package3d_urn="urn:adsk.eagle:package:23553/2" value="910"/>
 <part name="GND9" library="supply1" library_urn="urn:adsk.eagle:library:371" deviceset="GND" device=""/>
-<part name="R11" library="rcl" library_urn="urn:adsk.eagle:library:334" deviceset="R-EU_" device="R0805" package3d_urn="urn:adsk.eagle:package:23553/2" value="75R"/>
+<part name="R11" library="rcl" library_urn="urn:adsk.eagle:library:334" deviceset="R-EU_" device="R0805" package3d_urn="urn:adsk.eagle:package:23553/2" value="75"/>
 <part name="GND10" library="supply1" library_urn="urn:adsk.eagle:library:371" deviceset="GND" device=""/>
 <part name="GND11" library="supply1" library_urn="urn:adsk.eagle:library:371" deviceset="GND" device=""/>
@@
 <part name="R14" library="rcl" library_urn="urn:adsk.eagle:library:334" deviceset="R-EU_" device="R0805" package3d_urn="urn:adsk.eagle:package:23553/2" value="75R"/>
 <part name="GND24" library="supply1" library_urn="urn:adsk.eagle:library:371" deviceset="GND" device=""/>
-<part name="R15" library="rcl" library_urn="urn:adsk.eagle:library:334" deviceset="R-EU_" device="R0805" package3d_urn="urn:adsk.eagle:package:23553/2" value="10k"/>
-<part name="R16" library="rcl" library_urn="urn:adsk.eagle:library:334" deviceset="R-EU_" device="R0805" package3d_urn="urn:adsk.eagle:package:23553/2" value="10k"/>
+<part name="R15" library="rcl" library_urn="urn:adsk.eagle:library:334" deviceset="R-EU_" device="R0805" package3d_urn="urn:adsk.eagle:package:23553/2" value="1.1k"/>
+<part name="R16" library="rcl" library_urn="urn:adsk.eagle:library:334" deviceset="R-EU_" device="R0805" package3d_urn="urn:adsk.eagle:package:23553/2" value="510"/>
 <part name="GND25" library="supply1" library_urn="urn:adsk.eagle:library:371" deviceset="GND" device=""/>
 <part name="GND26" library="supply1" library_urn="urn:adsk.eagle:library:371" deviceset="GND" device=""/>
@@
 <text x="-2.54" y="-114.3" size="1.778" layer="98">PALSEL1</text>
 <text x="-2.54" y="-124.46" size="1.778" layer="98">PALSEL0</text>
+<text x="81.28" y="-114.3" size="1.778" layer="94" rot="R90">EXT LSB ADDRESS DATA</text>
 </plain>
 <instances>
@@
 </instance>
 <instance part="R10" gate="G$1" x="134.62" y="-114.3" smashed="yes">
-<attribute name="NAME" x="135.89" y="-110.2614" size="1.778" layer="95" rot="R180"/>
-<attribute name="VALUE" x="135.89" y="-117.602" size="1.778" layer="96" rot="R180"/>
+<attribute name="NAME" x="136.82" y="-108.8614" size="1.778" layer="95" rot="R180"/>
+<attribute name="VALUE" x="136.87" y="-111.002" size="1.778" layer="96" rot="R180"/>
 </instance>
 <instance part="GND9" gate="1" x="127" y="-114.3" smashed="yes" rot="R270">
@@
 </instance>
 <instance part="R11" gate="G$1" x="134.62" y="-101.6" smashed="yes">
-<attribute name="NAME" x="133.35" y="-100.1014" size="1.778" layer="95"/>
-<attribute name="VALUE" x="133.35" y="-104.902" size="1.778" layer="96"/>
+<attribute name="NAME" x="132.38" y="-97.3514" size="1.778" layer="95"/>
+<attribute name="VALUE" x="132.29" y="-99.702" size="1.778" layer="96"/>
 </instance>
 <instance part="GND10" gate="1" x="127" y="-106.68" smashed="yes" rot="R270">

Commit message: Add files via upload
Parts:
- added JP5: VRAM_A10, pinhead:PINHD-1X1
- added JP6: VRAMCS, pinhead:PINHD-1X1
- C1, C10, C16, C18, C19, C2, C20, C21, C28, C29, C3, C30, C31, C32, C33, C34, C35, C4, C6, C7, C9: value 0,1uF -> 0.1uF; device SnapEDA-Library:CAP -> rcl_my:C-EUC0805
- C11: value 220uF -> 1uF; device SnapEDA-Library:ELCAP -> rcl_my:C-EUC0805
- C12, C13: value 220uF -> 0.1uF; device SnapEDA-Library:ELCAP -> rcl_my:C-EUC0805
- C14: value 220uF -> 22uF; device SnapEDA-Library:ELCAP -> rcl_my:CPOL-EU153CLV-0505
- C15, C17: value 0,1uF -> 1uF; device SnapEDA-Library:CAP -> rcl_my:C-EUC0805
- C22, C23, C24, C25, C26, C27: value 1uF -> 0.1uF; device SnapEDA-Library:CAP -> rcl_my:C-EUC0805
- C36, C37, C38: value 0,1uF -> 1000; device SnapEDA-Library:CAP -> rcl_my:C-EUC0805
- C39: value 1nF -> 1000; device SnapEDA-Library:CAP -> rcl_my:C-EUC0805
- C40, C41, C42: value 1nF -> 0.1uF; device SnapEDA-Library:CAP -> rcl_my:C-EUC0805
- C43: value 22uF -> 0.1uF; device SnapEDA-Library:ELCAP -> rcl_my:C-EUC0805
- C44, C46, C47: value 22uF -> 220uF; device SnapEDA-Library:ELCAP -> rcl_my:CPOL-EU153CLV-0505
- C45: value 0,1uF -> 220uF; device SnapEDA-Library:CAP -> rcl_my:CPOL-EU153CLV-0505
- C5, C8: value 0,1uF -> 22uF; device SnapEDA-Library:CAP -> rcl_my:CPOL-EU153CLV-0505
- R29: value 75R -> 110
Connections:
- removed net N$61: C3.P$2, U4.VREF
- new net N$1: C44.+, R21.1
- new net N$28: C46.+, R19.1
- new net N$29: C47.+, R18.1
- new net N$30: C41.1, U4.VREF
- new net N$6: C5.+
- new net N$8: C45.+, R20.1
- net +1V2: now also C13.1, C14.+, C32.1, C33.1, C34.1, C35.1; no longer C21.P$2, C24.P$2, C25.P$2, C26.P$2, C27.P$2
- net +3V3: now also C1.2, C12.1, C19.1, C3.2, C7.1; no longer C10.P$1, C16.P$2, C20.P$2, C6.P$2
- net +5V: now also C2.1, C20.2, C4.1, C6.1, C8.+, C9.1; no longer C17.P$2, C18.P$2, C43.1, C44.1, C7.P$2, C8.P$2
- net AVCC: now also C10.1, C11.1, C41.2, C42.2, C43.1; no longer C15.P$2, C19.P$2, C3.P$1, C4.P$1
- net EXT_CLK: now also C39.1; no longer C39.P$2
- net GND: now also C10.2, C11.2, C12.2, C13.2, C15.2, C16.2, C17.2, C18.2, C19.2, C36.2, C37.2, C38.2, C5.-, C6.2, C7.2, C8.-, C9.2; no longer C40.P$1, C41.P$1, C42.P$1
- net N$11: now also C45.-; no longer C12.2
- net N$17: now also C46.-; no longer C13.2
- net N$19: now also C47.-; no longer C14.2
- net N$25: now also C39.2; no longer C39.P$1
- net N$27: now also C37.1; no longer C42.P$2
- net N$4: now also C44.-; no longer C11.2
- net N$62: now also C42.1; no longer C4.P$2
- net VAA@3: now also C40.1; no longer C5.P$2
- net VCC3.1: now also C21.1, C22.1, C23.1, C24.1, C25.1, C26.1, C27.1, C28.1, C29.1, C30.1, C31.1; no longer C28.P$2, C29.P$2, C30.P$2, C31.P$2, C32.P$2, C33.P$2, C34.P$2, C35.P$2, C36.P$2, C37.P$2, C38.P$2
- net VCC3.7: now also C36.1, C38.1; no longer C40.P$2, C41.P$2
- net VPPL1: now also C17.1, C18.1; no longer C2.P$2, C23.P$2
- net VPPL2: now also C15.1, C16.1; no longer C1.P$2, C22.P$2
- net VRAMCS: now also JP6.1
- net VRAM_A10: now also JP5.1
Other:
- moved on the sheet: C11, C12, C13, C43, Q2, R30, U7

Commit message: Add files via upload
Parts:
- C11: value 1uF -> 22uF
- C20: value 0.1uF -> 10uF
- JP4: value (none) -> A
Connections:
- new net VPLL1: U8.PLL1_VCCA, U8.PLL1_VCCD
- new net VPLL2: U8.PLL2_VCCA, U8.PLL2_VCCD
- net VCC3.1: now also U8.VCCIO1@1, U8.VCCIO1@2, U8.VCCIO1@3, U8.VCCIO2@1, U8.VCCIO2@2, U8.VCCIO2@3, U8.VCCIO3@1, U8.VCCIO3@2, U8.VCCIO3@3, U8.VCCIO4@1, U8.VCCIO4@2, U8.VCCIO4@3; no longer U8.VCC@1, U8.VCC@10, U8.VCC@11, U8.VCC@12, U8.VCC@13, U8.VCC@15, U8.VCC@16, U8.VCC@18, U8.VCC@2, U8.VCC@20, U8.VCC@3, U8.VCC@5, U8.VCC@6, U8.VCC@8
- net VPPL1: now also C15.1, C16.1, L1.1; no longer C17.1, C18.1, L2.2, U8.VPLL1
- net VPPL2: now also C17.1, C18.1, L2.2; no longer C15.1, C16.1, L1.1, U8.VPLL2
Other:
- note added: "EXT LSB CHR ADDRESS DATA"
- note removed: "EXT LSB ADDRESS DATA"
