File: PCB/FPGA_PPU.sch (EAGLE design)
At the start: 105 parts, among them CON1 DIP40, J1 J-08-SIP-100, T1 BC847, U1 SN74LVC8T245, U2 SN74LVC8T245, U3 SN74LVC541A, U4 ADV7125KST140, U5 THS7374IPWR, U6 EPCS4, U7 SN74LVC1G17DBVR, U8 EP2C5T144, X1 057-010-1

Commit message: Add files via upload
Parts:
- removed R30: 100k, rcl:R-EU_R0805
- added JP7: PALSEL0, jumper:JP4QE
- added JP8: PALSEL1, jumper:JP4QE
- added JP9: ALE EN, jumper:JP4QE
- added R7: 10k, rcl:R-EU_R0805
- added R8: 75R, rcl:R-EU_R0805
- C25, C27, C33, C34: value 0.1uF -> 1uF
- JP2: device jumper:JP4QE -> jumper:JP6QE
- JP3: value (none) -> NTSC/PAL; device jumper:JP6QE -> jumper:JP4QE
- JP4: value A -> (none); device jumper:JP1E -> jumper:JP4QE
- LED1: value (none) -> GNL-1206YC
- R1, R2: value 1k -> 100
- R10: value 910 -> 1k
- R11: value 75 -> 1k
- R12, R13, R14: value 75R -> 10k
- R15: value 1.1k -> 10k
- R16: value 510 -> 1k
- R17: value 10k -> 100k
- R18: value 75R -> 75
- R19: value 75R -> 910
- R23: value 75R -> 1.1k
- R24: value 100R -> 510
- R26, R27, R28, R9: value 10k -> 75R
- R29: value 110 -> 75R
- R3: value 1k -> 1k2
- U1: value SN74LVC8T245 -> EP2C5T144; device SnapEDA-Library:SN74LVC8T245 -> EP2C5T144:EP2C5T144
- U3: value SN74LVC541A -> SN74LVC8T245; device SnapEDA-Library:SN74LVC541A -> SnapEDA-Library:SN74LVC8T245
- U4: value ADV7125KST140 -> SN74LVC541A; device SnapEDA-Library:ADV7125KST140 -> SnapEDA-Library:SN74LVC541A
- U5: value THS7374IPWR -> SN74LVC1G17DBVR; device THS7374IPWR:THS7374IPWR -> SN74LVC1G17DBVR:SN74LVC1G17DBVR
- U7: value SN74LVC1G17DBVR -> ADV7125KST140; device SN74LVC1G17DBVR:SN74LVC1G17DBVR -> SnapEDA-Library:ADV7125KST140
- U8: value EP2C5T144 -> THS7374IPWR; device altera-cyclone-II:EP2C5T144 -> THS7374IPWR:THS7374IPWR
Connections:
- net VCC3.7 renamed N$6
- removed net +1V2: C13.1, C14.+, C32.1, C33.1, C34.1, C35.1, L1.2, L2.1, U8.VCCINT@1, U8.VCCINT@2, U8.VCCINT@3, U8.VCCINT@4, VR3.VOUT
- removed net +3V3: C1.2, C12.1, C19.1, C3.2, C7.1, L3.1, L4.1, LED1.A, R2.1, R25.1, R26.1, R27.1, R28.1, R3.1, R4.2, R5.2, R6.2, U1.VCCA, U2.VCCA, U3.VCC, U6.VCC@1, U6.VCC@2, U6.VCC@3, U7.VCC, VR1.VOUT, VR3.VIN, X1-4.S
- removed net ALE_FPGA: JP2-4.1, JP4.2, R28.2, U8.IO27
- removed net DATAO: U6.ASDI, U8.DATA0
- removed net GND8: R16.2, U3.A7, U3.A8, U3.GND
- removed net GND@8: U4.GND@1, U4.GND@2, U4.GND@3, U4.GND@4, U4.GND@5, U4.GND@6, U4.GND@7, U4.GND@8
- removed net N$10: JP3-4.2, U8.IO80
- removed net N$12: JP3-5.2, U8.IO79
- removed net N$13: JP3-6.2, U8.IO76
- removed net N$14: JP2-1.1, R25.2, U8.IO31
- removed net N$15: JP2-2.1, R26.2, U8.IO30
- removed net N$16: JP2-3.1, R27.2, U8.IO28
- removed net N$20: R4.1, U8.NSTATUS
- removed net N$21: R5.1, U8.NCONFIG
- removed net N$22: R6.1, U8.CONF_DONE
- removed net N$34: R22.1, U8.IO73
- removed net N$36: R23.1, U8.IO75
- removed net N$6 (its old number): C5.+
- removed net N$9: JP3-3.2, U8.IO81
- removed net VAA@3: C40.1, U4./BLANK, U4./PSAVE, U4.VAA@1, U4.VAA@2, U4.VAA@3
- removed net VCC3.1: C21.1, C22.1, C23.1, C24.1, C25.1, C26.1, C27.1, C28.1, C29.1, C30.1, C31.1, U8.VCCIO1@1, U8.VCCIO1@2, U8.VCCIO1@3, U8.VCCIO2@1, U8.VCCIO2@2, U8.VCCIO2@3, U8.VCCIO3@1, U8.VCCIO3@2, U8.VCCIO3@3, U8.VCCIO4@1, U8.VCCIO4@2, U8.VCCIO4@3
- removed net VRAMCS_FPGA: U3.Y2, U8.IO134
- new net CONF_DONE: R12.2, U1.CONF_DONE
- new net DATA0: U1.DATA0, U6.ASDI
- new net J0: JP2-1.2, U1.IO48
- new net J1: JP2-2.2, U1.IO47
- new net J2: JP2-3.2, U1.IO46
- new net J3: JP2-4.2, U1.IO45
- new net J4: JP2-5.2, U1.IO44
- new net J5: JP2-6.2, U1.IO43
- new net J6: JP4-1.2, JP9-1.1, R7.2, U1.IO11
- new net NCE: R15.1, U1.NCE
- new net NCONFIG: R14.1, U1.NCONFIG
- new net NSTATUS: R13.1, U1.NSTATUS
- new net NTSC/PAL: JP3-1.2, R4.2, U1.IO14
- new net PALSEL0: JP7-1.2, R5.2, U1.IO12
- new net PALSEL1: JP8-1.2, R6.2, U1.IO13
- new net VCCINT: C13.1, C14.+, C25.2, C27.2, C33.1, C34.1, L1.2, L2.1, U1.VCCINT@1, U1.VCCINT@2, U1.VCCINT@3, U1.VCCINT@4, VR3.VOUT
- new net VCCIO: C1.2, C12.1, C19.1, C21.2, C22.2, C23.2, C24.2, C26.2, C28.2, C29.1, C3.2, C30.1, C31.1, C32.1, C35.1, C7.1, L3.1, L4.1, LED1.A, R10.2, R11.2, R12.1, R13.2, R14.2, R4.1, R5.1, R6.1, R7.1, U1.VCCIO1@1, U1.VCCIO1@2, U1.VCCIO1@3, U1.VCCIO2@1, U1.VCCIO2@2, U1.VCCIO2@3, U1.VCCIO3@1, U1.VCCIO3@2, U1.VCCIO3@3, U1.VCCIO4@1, U1.VCCIO4@2, U1.VCCIO4@3, U2.VCCA, U3.VCCA, U4.VCC, U5.VCC, U6.VCC@1, U6.VCC@2, U6.VCC@3, VR1.VOUT, VR3.VIN, X1-4.S
- new net VRCS_FPGA: U1.IO73, U4.Y2
- net +5V: now also C2.2, C4.2, C5.+, U3.VCCB@1, U3.VCCB@2; no longer C2.1, C4.1, U1.VCCB@1, U1.VCCB@2
- net /CSO: now also U1.IO2(/CSO); no longer U8.IO2(/CSO)
- net /DBE: now also U4.A6; no longer U3.A6
- net /DBE_FPGA: now also U1.IO60, U3./OE, U4.Y6; no longer U2./OE, U3.Y6, U8.IO113
- net /PRD: now also U1.IO65, U2.DIR; no longer U1.DIR, U8.IO120
- net /PWR: now also U1.IO59; no longer U8.IO112
- net A0: now also U4.A5; no longer U3.A5
- net A0_FPGA: now also U1.IO61, U4.Y5; no longer U3.Y5, U8.IO114
- net A1: now also U4.A4; no longer U3.A4
- net A1_FPGA: now also U1.IO62, U4.Y4; no longer U3.Y4, U8.IO115
- net A2: now also U4.A3; no longer U3.A3
- net A2_FPGA: now also U1.IO63, U4.Y3; no longer U3.Y3, U8.IO118
- net ALE: now also JP9-1.2; no longer JP4.1
- net ASDO: now also U1.IO1(ASDO); no longer U8.IO1(ASDO)
- net AVCC: now also C40.1, R25.2, U7./BLANK, U7./PSAVE, U7.VAA@1, U7.VAA@2, U7.VAA@3, U8.VS+; no longer R17.2, U5.VS+
- net B0: now also U1.IO23, U7.B0; no longer U4.B0, U8.IO48
- net B1: now also U1.IO22, U7.B1; no longer U4.B1, U8.IO47
- net B2: now also U1.IO21, U7.B2; no longer U4.B2, U8.IO45
- net B3: now also U1.IO20, U7.B3; no longer U4.B3, U8.IO44
- net B4: now also U1.IO19, U7.B4; no longer U4.B4, U8.IO43
- net B5: now also U1.IO18, U7.B5; no longer U4.B5, U8.IO42
- net B6: now also U1.IO17, U7.B6; no longer U4.B6, U8.IO41
- net B7: now also U1.IO16, U7.B7; no longer U4.B7, U8.IO40
- net CLK0: now also U1.CLK0; no longer U8.CLK0
- net CLK4: now also U1.CLK4; no longer U8.CLK4
- net CLK6: now also U1.CLK6; no longer U8.CLK6
- net CLK7: now also U1.CLK7, U5.Y; no longer U7.Y, U8.CLK7
- net D0_FPGA: now also U1.IO10, U3.A0; no longer U2.A0, U8.IO26
- net D1_FPGA: now also U1.IO9, U3.A1; no longer U2.A1, U8.IO25
- net D2_FPGA: now also U1.IO8, U3.A2; no longer U2.A2, U8.IO24
- net D3_FPGA: now also U1.IO7, U3.A3; no longer U2.A3, U8.IO9
- net D4_FPGA: now also U1.IO6, U3.A4; no longer U2.A4, U8.IO8
- net D5_FPGA: now also U1.IO5, U3.A5; no longer U2.A5, U8.IO7
- net D6_FPGA: now also U1.IO4, U3.A6; no longer U2.A6, U8.IO4
- net D7_FPGA: now also U1.IO3, U3.A7; no longer U2.A7, U8.IO3
- net DAC_CLK: now also R18.1, U1.IO15; no longer R11.1, U8.IO32
- net DB0: now also U3.B0; no longer U2.B0
- net DB1: now also U3.B1; no longer U2.B1
- net DB2: now also U3.B2; no longer U2.B2
- net DB3: now also U3.B3; no longer U2.B3
- net DB4: now also U3.B4; no longer U2.B4
- net DB5: now also U3.B5; no longer U2.B5
- net DB6: now also U3.B6; no longer U2.B6
- net DB7: now also U3.B7; no longer U2.B7
- net DCLK: now also U1.DCLK; no longer U8.DCLK
- net G0: now also U1.IO31, U7.G0; no longer U4.G0, U8.IO60
- net G1: now also U1.IO30, U7.G1; no longer U4.G1, U8.IO59
- net G2: now also U1.IO29, U7.G2; no longer U4.G2, U8.IO58
- net G3: now also U1.IO28, U7.G3; no longer U4.G3, U8.IO57
- net G4: now also U1.IO27, U7.G4; no longer U4.G4, U8.IO55
- net G5: now also U1.IO26, U7.G5; no longer U4.G5, U8.IO53
- net G6: now also U1.IO25, U7.G6; no longer U4.G6, U8.IO52
- net G7: now also U1.IO24, U7.G7; no longer U4.G7, U8.IO51
- net GND: now also C1.1, C14.-, C2.1, C20.1, C21.1, C22.1, C23.1, C24.1, C25.1, C26.1, C27.1, C28.1, C29.2, C3.1, C30.2, C31.2, C32.2, C33.2, C34.2, C35.2, C4.1, C40.2, C43.2, JP2-1.1, JP2-2.1, JP2-3.1, JP2-4.1, JP2-5.1, JP2-6.1, JP4-1.1, JP7-1.1, JP8-1.1, R15.2, R16.2, R17.2, R19.1, R20.1, R21.1, R22.1, R24.2, R3.2, U1.GAPLL1, U1.GAPLL2, U1.GND@10, U1.GND@11, U1.GND@12, U1.GND@13, U1.GND@14, U1.GND@18, U1.GND@19, U1.GND@20, U1.GND@21, U1.GND@22, U1.GND@23, U1.GND@7, U1.GND@8, U1.GND@9, U1.GPLL1@1, U1.GPLL1@2, U1.GPLL2@1, U1.GPLL2@2, U1.MSEL0, U1.MSEL1, U3.GND@1, U3.GND@2, U3.GND@3, U4./OE1, U4./OE2, U4.A7, U4.A8, U4.GND, U7./IOB, U7./IOG, U7./IOR, U7./SYNC, U7.GND@1, U7.GND@2, U7.GND@3, U7.GND@4, U7.GND@5, U7.GND@6, U7.GND@7, U7.GND@8, U8.DISABLE, U8.GND, VR1.GND, VR2.GND, VR3.GND; no longer JP2-1.2, JP2-2.2, JP2-3.2, JP2-4.2, JP3-2.1, JP3-3.1, JP3-4.1, JP3-5.1, JP3-6.1, R1.1, R10.1, R12.1, R13.1, R14.1, R29.2, R30.2, R9.2, U3./OE1, U3./OE2, U4./IOB, U4./IOG, U4./IOR, U4./SYNC, U5.DISABLE, U7.GND, U8.GND@1, U8.GND@10, U8.GND@11, U8.GND@12, U8.GND@13, U8.GND@14, U8.GND@15, U8.GND@16, U8.GND@17, U8.GND@18, U8.GND@19, U8.GND@2, U8.GND@20, U8.GND@21, U8.GND@22, U8.GND@23, U8.GND@3, U8.GND@4, U8.GND@5, U8.GND@6, U8.GND@7, U8.GND@8, U8.GND@9, U8.MSEL0, U8.MSEL1
- net HSYNC: now also R9.2; no longer R23.2
- net INT_FPGA: now also R2.2, U1.IO50; no longer R24.2, U8.IO93
- net N$1: now also R26.1; no longer R21.1
- net N$18: now also R22.2, U7.IOB, U8.CH3_IN; no longer R12.2, U4.IOB, U5.CH3_IN
- net N$2: now also R8.1, U1.IO40; no longer JP3-1.2, U8.IO87
- net N$23: now also R21.2, U7.IOG, U8.CH2_IN; no longer R13.2, U4.IOG, U5.CH2_IN
- net N$24: now also R2.1; no longer R24.1
- net N$25: now also R17.1, U5.A; no longer R30.1, U7.A
- net N$26: now also R3.1; no longer R29.1
- net N$28: now also R28.1; no longer R19.1
- net N$29: now also R29.1; no longer R18.1
- net N$30: now also U7.VREF; no longer U4.VREF
- net N$5: now also R9.1, U1.IO42; no longer JP3-2.2, U8.IO86
- net N$58: now also R19.2, U7.RSET; no longer R10.2, U4.RSET
- net N$59: now also R18.2, U7.CLK; no longer R11.2, U4.CLK
- net N$62: now also U7.COMP; no longer U4.COMP
- net N$65: now also R20.2, U7.IOR, U8.CH1_IN; no longer R14.2, U4.IOR, U5.CH1_IN
- net N$66: now also R23.2, R24.1, U8.CH4_IN; no longer R15.2, R16.1, U5.CH4_IN
- net N$67: now also R25.1, U8.BYPASS; no longer R17.1, U5.BYPASS
- net N$69: now also R29.2, U8.CH4_OUT; no longer R18.2, U5.CH4_OUT
- net N$7: now also JP5.1, R1.1; no longer R9.1, U8.NCE
- net N$70: now also R28.2, U8.CH3_OUT; no longer R19.2, U5.CH3_OUT
- net N$71: now also R27.2, U8.CH2_OUT; no longer R20.2, U5.CH2_OUT
- net N$72: now also R26.2, U8.CH1_OUT; no longer R21.2, U5.CH1_OUT
- net N$8: now also R27.1; no longer R20.1
- net PA0: now also U1.IO51; no longer U8.IO94
- net PA1: now also U1.IO52; no longer U8.IO96
- net PA10: now also U1.IO69; no longer U8.IO126
- net PA11: now also U1.IO68; no longer U8.IO125
- net PA12: now also U1.IO67; no longer U8.IO122
- net PA13: now also U1.IO66; no longer U8.IO121
- net PA2: now also U1.IO53; no longer U8.IO97
- net PA3: now also U1.IO54; no longer U8.IO99
- net PA4: now also U1.IO55; no longer U8.IO100
- net PA5: now also U1.IO56; no longer U8.IO101
- net PA6: now also U1.IO57; no longer U8.IO103
- net PA7: now also U1.IO58; no longer U8.IO104
- net PA8: now also U1.IO71; no longer U8.IO132
- net PA9: now also U1.IO70; no longer U8.IO129
- net PD0: now also U2.B0; no longer U1.B0
- net PD0_FPGA: now also U1.IO81, U2.A0; no longer U1.A0, U8.IO144
- net PD1: now also U2.B1; no longer U1.B1
- net PD1_FPGA: now also U1.IO80, U2.A1; no longer U1.A1, U8.IO143
- net PD2: now also U2.B2; no longer U1.B2
- net PD2_FPGA: now also U1.IO79, U2.A2; no longer U1.A2, U8.IO142
- net PD3: now also U2.B3; no longer U1.B3
- net PD3_FPGA: now also U1.IO78, U2.A3; no longer U1.A3, U8.IO141
- net PD4: now also U2.B4; no longer U1.B4
- net PD4_FPGA: now also U1.IO77, U2.A4; no longer U1.A4, U8.IO139
- net PD5: now also U2.B5; no longer U1.B5
- net PD5_FPGA: now also U1.IO76, U2.A5; no longer U1.A5, U8.IO137
- net PD6: now also U2.B6; no longer U1.B6
- net PD6_FPGA: now also U1.IO75, U2.A6; no longer U1.A6, U8.IO136
- net PD7: now also U2.B7; no longer U1.B7
- net PD7_FPGA: now also U1.IO74, U2.A7; no longer U1.A7, U8.IO135
- net PD_OE: now also U1.IO72, U2./OE; no longer U1./OE, U8.IO133
- net R0: now also U1.IO39, U7.R0; no longer U4.R0, U8.IO72
- net R1: now also U1.IO38, U7.R1; no longer U4.R1, U8.IO71
- net R2: now also U1.IO37, U7.R2; no longer U4.R2, U8.IO70
- net R3: now also U1.IO36, U7.R3; no longer U4.R3, U8.IO69
- net R4: now also U1.IO35, U7.R4; no longer U4.R4, U8.IO67
- net R5: now also U1.IO34, U7.R5; no longer U4.R5, U8.IO65
- net R6: now also U1.IO33, U7.R6; no longer U4.R6, U8.IO64
- net R7: now also U1.IO32, U7.R7; no longer U4.R7, U8.IO63
- net RW: now also U4.A1; no longer U3.A1
- net RW_FPGA: now also U1.IO64, U3.DIR, U4.Y1; no longer U2.DIR, U3.Y1, U8.IO119
- net SYNC_FPGA: now also R23.1, U1.IO41; no longer R15.1, U8.IO74
- net TCK: now also R16.1, U1.TCK; no longer R1.2, U8.TCK
- net TDI: now also R10.1, U1.TDI; no longer R3.2, U8.TDI
- net TDO: now also U1.TDO; no longer U8.TDO
- net TMS: now also R11.1, U1.TMS; no longer R2.2, U8.TMS
- net VPLL1: now also C15.1, C16.1, L1.1; no longer U8.PLL1_VCCA, U8.PLL1_VCCD
- net VPLL2: now also C17.1, C18.1, L2.2; no longer U8.PLL2_VCCA, U8.PLL2_VCCD
- net VPPL1: now also U1.VAPLL1, U1.VPLL1; no longer C15.1, C16.1, L1.1
- net VPPL2: now also U1.VAPLL2, U1.VPLL2; no longer C17.1, C18.1, L2.2
- net VRAMCS: now also U4.A2; no longer U3.A2
- net VRAM_A10: now also R1.2, U1.IO49; no longer JP5.1, U8.IO92
- net VSYNC: now also R8.2; no longer R22.2
Other:
- note removed: "NTSC/PAL"
- note removed: "PALSEL0"
- note removed: "PALSEL1"
- moved on the sheet: C1, C10, C11, C12, C13, C14, C15, C16, C17, C18, C19, C2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

Commit message: Add files via upload
Parts:
- R2: value 100 -> 1k
Changed lines of the file:
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@@
 <?xml version="1.0" encoding="utf-8"?>
 <!DOCTYPE eagle SYSTEM "eagle.dtd">
-<eagle version="9.6.2">
+<eagle version="9.4.2">
 <drawing>
 <settings>
@@
 <part name="GND29" library="supply1" library_urn="urn:adsk.eagle:library:371" deviceset="GND" device=""/>
 <part name="R9" library="rcl" library_urn="urn:adsk.eagle:library:334" deviceset="R-EU_" device="R0805" package3d_urn="urn:adsk.eagle:package:23553/2" value="75R"/>
-<part name="R2" library="rcl" library_urn="urn:adsk.eagle:library:334" deviceset="R-EU_" device="R0805" package3d_urn="urn:adsk.eagle:package:23553/2" value="100"/>
+<part name="R2" library="rcl" library_urn="urn:adsk.eagle:library:334" deviceset="R-EU_" device="R0805" package3d_urn="urn:adsk.eagle:package:23553/2" value="1k"/>
 <part name="GND30" library="supply1" library_urn="urn:adsk.eagle:library:371" deviceset="GND" device=""/>
 <part name="R4" library="rcl" library_urn="urn:adsk.eagle:library:334" deviceset="R-EU_" device="R0805" package3d_urn="urn:adsk.eagle:package:23553/2" value="10k"/>
